Commit message: Update sawyer simulation files

File: examples/examples_files/sawyer_arm.urdf (robot description, URDF)
Before this commit: robot sawyer, 11 links, 10 joints
Links:
- removed link base
- removed link head
- removed link pedestal
Joints:
- removed joint head_pan
- removed joint pedestal_fixed
- removed joint right_arm_mount

Commit message: Update sawyer meshs

File: examples/examples_files/sawyer_arm.urdf (robot description, URDF)
Before this commit: robot sawyer, 8 links, 7 joints
Links:
- link right_arm_base_link: geometry collision cylinder length=0.24 radius=0.08; visual mesh filename=examples/examples_files/sawyer_mesh/base.DAE
- link right_l0: geometry collision sphere radius=0.07; visual mesh filename=examples/examples_files/sawyer_mesh/l0.DAE
- link right_l1: geometry collision sphere radius=0.07; visual mesh filename=examples/examples_files/sawyer_mesh/l1.DAE
- link right_l2: geometry collision cylinder length=0.34 radius=0.06; visual mesh filename=examples/examples_files/sawyer_mesh/l2.DAE
- link right_l3: geometry collision sphere radius=0.06; visual mesh filename=examples/examples_files/sawyer_mesh/l3.DAE
- link right_l4: geometry collision cylinder length=0.30 radius=0.045; visual mesh filename=examples/examples_files/sawyer_mesh/l4.DAE
- link right_l5: geometry collision sphere radius=0.06; visual mesh filename=examples/examples_files/sawyer_mesh/l5.DAE
- link right_l6: geometry collision cylinder length=0.05 radius=0.055; visual mesh filename=examples/examples_files/sawyer_mesh/l6.DAE
